File: hardware/gigafoc.sch (EAGLE design)
At the start: 96 parts, among them IC1 STSPIN233, IC2 STSPIN233, IC3 STSPIN233, IC4 STSPIN233, IC5 STSPIN233, IC6 LMR51450SDRRR, X1 ARDUINO_GIGA_R1_WIFI, X10 53261-06, X2 53261-04, X5 53261-06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

Commit message: snapshot
Parts:
- X1: value ARDUINO_GIGA_R1_WIFI -> 53261-04; device SparkFun-Boards:ARDUINO_GIGA_R1_WIFI -> con-molex:53261-04
- X10: value 53261-06 -> ARDUINO_GIGA_R1_WIFI; device con-molex:53261-06 -> SparkFun-Boards:ARDUINO_GIGA_R1_WIFI
- X2: value 53261-04 -> 53261-06; device con-molex:53261-04 -> con-molex:53261-06
- X3, X4: value (none) -> 53261-06; device con-amp-mt:S02P -> con-molex:53261-06
- X8, X9: value 53261-06 -> (none); device con-molex:53261-06 -> con-amp-mt:S02P
Connections:
- net 24V: now also X8-1.S; no longer X4-1.S
- net 3.3V: now also X1-4.S, X10.3.3V, X2-2.S, X3-2.S, X4-2.S; no longer X1.3.3V, X10-2.S, X2-4.S, X8-2.S, X9-2.S
- net 5V: now also X10.5V; no longer X1.5V
- net EN_M1: now also X10.2; no longer X1.2
- net EN_M2: now also X10.14; no longer X1.14
- net EN_M3: now also X10.0; no longer X1.0
- net EN_M4: now also X10.16; no longer X1.16
- net EN_M5: now also X10.17; no longer X1.17
- net FAULT_M1: now also X10.94; no longer X1.94
- net FAULT_M2: now also X10.93; no longer X1.93
- net FAULT_M3: now also X10.84; no longer X1.84
- net FAULT_M4: now also X10.A7; no longer X1.A7
- net FAULT_M5: now also X10.A6; no longer X1.A6
- net GND: now also X1-1.S, X10.GND, X3-1.S, X4-1.S, X8-2.S, X9-2.S; no longer X1.GND, X10-1.S, X3-2.S, X4-2.S, X8-1.S, X9-1.S
- net MAG_CS1: now also X10.56, X3-6.S; no longer X1.56, X6-6.S
- net MAG_CS2: now also X10.58, X4-6.S; no longer X1.58, X7-6.S
- net MAG_CS3: now also X10.60, X5-6.S; no longer X1.60, X8-6.S
- net MAG_CS4: now also X10.62, X6-6.S; no longer X1.62, X9-6.S
- net MAG_CS5: now also X10.64, X7-6.S; no longer X1.64, X10-6.S
- net MAG_MISO: now also X10.12, X3-4.S, X4-4.S, X5-4.S; no longer X1.12, X10-4.S, X8-4.S, X9-4.S
- net MAG_MOSI: now also X10.11, X3-3.S, X4-3.S, X5-3.S; no longer X1.11, X10-3.S, X8-3.S, X9-3.S
- net MAG_SCK: now also X10.13, X3-5.S, X4-5.S, X5-5.S; no longer X1.13, X10-5.S, X8-5.S, X9-5.S
- net MISO: now also X10.SPI1_CIPO, X2-4.S; no longer X1.SPI1_CIPO, X5-4.S
- net MOSI: now also X10.SPI1_COPI, X2-3.S; no longer X1.SPI1_COPI, X5-3.S
- net N$1: now also X10.75; no longer X1.75
- net N$10: now also X10.23; no longer X1.23
- net N$102: now also X10.!RESET; no longer X1.!RESET
- net N$103: now also X10.IOREF; no longer X1.IOREF
- net N$11: now also X10.55; no longer X1.55
- net N$12: now also X10.52; no longer X1.52
- net N$13: now also X10.50; no longer X1.50
- net N$14: now also X10.25; no longer X1.25
- net N$15: now also X10.46; no longer X1.46
- net N$16: now also X10.44; no longer X1.44
- net N$17: now also X10.42; no longer X1.42
- net N$18: now also X10.40; no longer X1.40
- net N$19: now also X10.74; no longer X1.74
- net N$2: now also X10.73; no longer X1.73
- net N$20: now also X10.72; no longer X1.72
- net N$21: now also X10.70; no longer X1.70
- net N$22: now also X10.68; no longer X1.68
- net N$23: now also X10.22; no longer X1.22
- net N$24: now also X10.24; no longer X1.24
- net N$25: now also X10.26; no longer X1.26
- net N$26: now also X10.27; no longer X1.27
- net N$27: now also X10.29; no longer X1.29
- net N$28: now also X10.31; no longer X1.31
- net N$29: now also X10.54; no longer X1.54
- net N$3: now also X10.71; no longer X1.71
- net N$30: now also X10.53; no longer X1.53
- net N$31: now also X10.51; no longer X1.51
- net N$32: now also X10.49; no longer X1.49
- net N$33: now also X10.47; no longer X1.47
- net N$34: now also X10.45; no longer X1.45
- net N$35: now also X10.43; no longer X1.43
- net N$36: now also X10.41; no longer X1.41
- net N$37: now also X10.39; no longer X1.39
- net N$38: now also X10.37; no longer X1.37
- net N$39: now also X10.35; no longer X1.35
- net N$4: now also X10.69; no longer X1.69
- net N$40: now also X10.33; no longer X1.33
- net N$44: now also X10.28; no longer X1.28
- net N$45: now also X10.30; no longer X1.30
- net N$46: now also X10.38; no longer X1.38
- net N$47: now also X10.36; no longer X1.36
- net N$48: now also X10.34; no longer X1.34
- net N$49: now also X10.32; no longer X1.32
- net N$5: now also X10.67; no longer X1.67
- net N$55: now also X10.SCL; no longer X1.SCL
- net N$56: now also X10.SDA; no longer X1.SDA
- net N$57: now also X10.19; no longer X1.19
- net N$59: now also X9-1.S; no longer X3-1.S
- net N$6: now also X10.65; no longer X1.65
- net N$7: now also X10.63; no longer X1.63
- net N$77: now also X10.AREF; no longer X1.AREF
- net N$8: now also X10.61; no longer X1.61
- net N$83: now also X10.A11; no longer X1.A11
- net N$84: now also X10.A10; no longer X1.A10
- net N$85: now also X10.A9; no longer X1.A9
- net N$86: now also X10.A8; no longer X1.A8
- net N$9: now also X10.59; no longer X1.59
- net SCK: now also X10.SPI1_SCK, X2-5.S; no longer X1.SPI1_SCK, X5-5.S
- net SCL1: now also X1-3.S, X10.SCL1; no longer X1.SCL1, X2-3.S
- net SDA1: now also X1-2.S, X10.SDA1; no longer X1.SDA1, X2-2.S
- net SENSE_M1: now also X10.A5; no longer X1.A5
- net SENSE_M2: now also X10.A4; no longer X1.A4
- net SENSE_M3: now also X10.A3; no longer X1.A3
- net SENSE_M4: now also X10.A1; no longer X1.A1
- net SENSE_M5: now also X10.A0; no longer X1.A0
- net U_M1: now also X10.10; no longer X1.10
- net U_M2: now also X10.85; no longer X1.85
- net U_M3: now also X10.7; no longer X1.7
- net U_M4: now also X10.6; no longer X1.6
- net U_M5: now also X10.4; no longer X1.4
- net VS: now also X10.VIN; no longer X1.VIN
- net V_M1: now also X10.1; no longer X1.1
- net V_M2: now also X10.66; no longer X1.66
- net V_M3: now also X10.5; no longer X1.5
- net V_M4: now also X10.8; no longer X1.8
- net V_M5: now also X10.15; no longer X1.15
- net W5500_CS: now also X10.18, X2-6.S; no longer X1.18, X5-6.S
- net W_M1: now also X10.57; no longer X1.57
- net W_M2: now also X10.3; no longer X1.3
- net W_M3: now also X10.A2; no longer X1.A2
- net W_M4: now also X10.9; no longer X1.9
- net W_M5: now also X10.48; no longer X1.48
Other:
- moved on the sheet: X2-1, X2-2, X2-3, X2-4, X5-1, X5-2, X5-3, X5-4, X5-5, X5-6, X6-1, X6-2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
